File: LED Driver 4x8 mux.sch (KiCad schematic (older format))
At the start: 22 parts, among them J1 Barrel_Jack_Switch, J3 8P8C_Shielded_x4

Commit message: update PCB
Parts:
- U1: renamed from U?; footprint D16 -> Custom Footprints:SN74LV138ATD; Manufacturer (none) -> Texas Instruments; Part # (none) -> SN74LV138ATD
- gave numbers to parts that had none: 12
Connections:
- net GND: no longer U1.7 (Y7)
- net IN8: now reaches U3.10 (4B), U3.9 (4A)
- net IN8: now also U1.7 (Y7)
Other:
- moved on the sheet: H1, H2, H3, H4

Commit message: PCB draft finished
Parts:
- PS1: footprint CONV_PXO7805-500-M-TR -> Custom Footprints:18V_to_5V_PXO7805-500-M-TR
Connections:
- net GND: now also J3.26, J3.28, J3.30, J3.32; no longer J3.10, J3.12, J3.14, J3.16
- net LED-: now also J3.10, J3.12, J3.14, J3.16; no longer J3.26, J3.28, J3.30, J3.32
- net LED1+: now also J3.1; no longer J3.25
- net LED2+: now also J3.3; no longer J3.27
- net LED3+: now also J3.5; no longer J3.29
- net LED4+: now also J3.7; no longer J3.31
- net LED5+: now also J3.9; no longer J3.1
- net LED6+: now also J3.11; no longer J3.3
- net LED7+: now also J3.13; no longer J3.5
- net LED8+: now also J3.15; no longer J3.7
- net OUT1: now also J3.25; no longer J3.9
- net OUT2: now also J3.27; no longer J3.11
- net OUT3: now also J3.29; no longer J3.13
- net Thermistor: now also J3.31; no longer J3.15
Other:
- moved on the sheet: J3A, J3B, J3D
Changed lines of the file:
@@
 L Custom_parts:8P8C_Shielded_x4 J3
 U 4 1 5F58DBB9
-P 7300 4050
-F 0 "J3" H 7400 4700 50  0000 R CNN
-F 1 "8P8C_Shielded_x4" H 7650 4600 50  0000 R CNN
-F 2 "Custom Footprints:RJ45_x4-RJSSE-5380-04" V 7300 4075 50  0001 C CNN
-F 3 "https://cdn.amphenol-icc.com/media/wysiwyg/files/drawing/rjsse538004.pdf" V 7300 4075 50  0001 C CNN
-F 4 "Amphenol ICC (Commercial Products)" H 7300 4050 50  0001 C CNN "Manufacturer"
-F 5 "RJSSE-5380-04" H 7300 4050 50  0001 C CNN "Part #"
-	4    7300 4050
-	-1   0    0    1
+P 1150 5000
+F 0 "J3" H 1250 5650 50  0000 R CNN
+F 1 "8P8C_Shielded_x4" H 1500 5550 50  0000 R CNN
+F 2 "Custom Footprints:RJ45_x4-RJSSE-5380-04" V 1150 5025 50  0001 C CNN
+F 3 "https://cdn.amphenol-icc.com/media/wysiwyg/files/drawing/rjsse538004.pdf" V 1150 5025 50  0001 C CNN
+F 4 "Amphenol ICC (Commercial Products)" H 1150 5000 50  0001 C CNN "Manufacturer"
+F 5 "RJSSE-5380-04" H 1150 5000 50  0001 C CNN "Part #"
+	4    1150 5000
+	1    0    0    1
 $EndComp
 $Comp
@@
 L Custom_parts:8P8C_Shielded_x4 J3
 U 2 1 5F589234
-P 1150 5000
-F 0 "J3" H 1250 5650 50  0000 R CNN
-F 1 "8P8C_Shielded_x4" H 1500 5550 50  0000 R CNN
-F 2 "Custom Footprints:RJ45_x4-RJSSE-5380-04" V 1150 5025 50  0001 C CNN
-F 3 "https://cdn.amphenol-icc.com/media/wysiwyg/files/drawing/rjsse538004.pdf" V 1150 5025 50  0001 C CNN
-F 4 "Amphenol ICC (Commercial Products)" H 1150 5000 50  0001 C CNN "Manufacturer"
-F 5 "RJSSE-5380-04" H 1150 5000 50  0001 C CNN "Part #"
-	2    1150 5000
-	1    0    0    1
+P 7300 6150
+F 0 "J3" H 7400 6800 50  0000 R CNN
+F 1 "8P8C_Shielded_x4" H 7650 6700 50  0000 R CNN
+F 2 "Custom Footprints:RJ45_x4-RJSSE-5380-04" V 7300 6175 50  0001 C CNN
+F 3 "https://cdn.amphenol-icc.com/media/wysiwyg/files/drawing/rjsse538004.pdf" V 7300 6175 50  0001 C CNN
+F 4 "Amphenol ICC (Commercial Products)" H 7300 6150 50  0001 C CNN "Manufacturer"
+F 5 "RJSSE-5380-04" H 7300 6150 50  0001 C CNN "Part #"
+	2    7300 6150
+	-1   0    0    1
 $EndComp
 $Comp
@@
 L Custom_parts:8P8C_Shielded_x4 J3
 U 1 1 5F5922AC
-P 7300 6150
-F 0 "J3" H 7350 6800 50  0000 R CNN
-F 1 "8P8C_Shielded_x4" H 7650 6700 50  0000 R CNN
-F 2 "Custom Footprints:RJ45_x4-RJSSE-5380-04" V 7300 6175 50  0001 C CNN
-F 3 "https://cdn.amphenol-icc.com/media/wysiwyg/files/drawing/rjsse538004.pdf" V 7300 6175 50  0001 C CNN
-F 4 "Amphenol ICC (Commercial Products)" H 7300 6150 50  0001 C CNN "Manufacturer"
-F 5 "RJSSE-5380-04" H 7300 6150 50  0001 C CNN "Part #"
-	1    7300 6150
+P 7300 4050
+F 0 "J3" H 7350 4700 50  0000 R CNN
+F 1 "8P8C_Shielded_x4" H 7650 4600 50  0000 R CNN
+F 2 "Custom Footprints:RJ45_x4-RJSSE-5380-04" V 7300 4075 50  0001 C CNN
+F 3 "https://cdn.amphenol-icc.com/media/wysiwyg/files/drawing/rjsse538004.pdf" V 7300 4075 50  0001 C CNN
+F 4 "Amphenol ICC (Commercial Products)" H 7300 4050 50  0001 C CNN "Manufacturer"
+F 5 "RJSSE-5380-04" H 7300 4050 50  0001 C CNN "Part #"
+	1    7300 4050
 	-1   0    0    1
 $EndComp
@@
 F 0 "PS1" H 3625 3115 50  0000 C CNN
 F 1 "PXO7805-500-M-TR" H 3625 3024 50  0000 C CNN
-F 2 "CONV_PXO7805-500-M-TR" H 3100 2550 50  0001 L BNN
+F 2 "Custom Footprints:18V_to_5V_PXO7805-500-M-TR" H 3100 2550 50  0001 L BNN
 F 3 "https://www.cui.com/product/resource/pxo78-500-m.pdf" H 3700 2850 50  0001 L BNN
 F 4 "CUI Inc." H 3600 2850 50  0001 C CNN "Manufacturer"

Commit message: Add thermistor breakout
Parts:
- added J2: Conn_01x02_Female, Connector_Wire:SolderWire-0.5sqmm_1x02_P4.6mm_D0.9mm_OD2.1mm, symbol Connector:Conn_01x02_Female
- added JP1: Jumper_NO_Small, Jumper:SolderJumper-2_P1.3mm_Open_TrianglePad1.0x1.5mm, symbol Device:Jumper_NO_Small
- U2, U3: value MIC4467YWM-TR -> TC4468EOE
- renumbered C3 to C2, C2 to C3
Connections:
- net GND: now also J2.2 (Pin_2)
- net Thermistor: now also JP1.1
- new net: J2.1 (Pin_1), JP1.2
Other:
- moved on the sheet: C1, C2, C3, C4, C5, H1, H2, H3, H4, J1, J3A, J3B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

Commit message: Board powered off LED river backup
Parts:
- removed J1: Barrel_Jack_Switch, Custom Footprints:DC-jack_54-00165, symbol Connector:Barrel_Jack_Switch
- removed JP1: Jumper_NO_Small, Jumper:SolderJumper-2_P1.3mm_Open_TrianglePad1.0x1.5mm, symbol Device:Jumper_NO_Small
- J1: renamed from J2; value Conn_01x02_Female -> 8P8C_Shielded_x4; footprint Connector_Wire:SolderWire-0.5sqmm_1x02_P4.6mm_D0.9mm_OD2.1mm -> Custom Footprints:RJ45_x4-RJSSE-5380-04
- renumbered J3 to J2, Q4 to Q1, Q3 to Q2, Q2 to Q3, Q1 to Q4, U3 to U2, U2 to U3
Connections:
- net +18V is gone; now on net LED+: C1.1, C4.2, C5.2, PS1.1 (+Vin), U2.15 (VDD), U2.16 (VDD), U3.15 (VDD), U3.16 (VDD)
- net Thermistor: now also J1.1 (Pin_1)
Changed lines of the file:
@@
 $EndComp
 $Comp
-L Custom_parts:8P8C_Shielded_x4 J3
+L Custom_parts:8P8C_Shielded_x4 J2
 U 4 1 5F58DBB9
 P 1150 5000
-F 0 "J3" H 1250 5650 50  0000 R CNN
+F 0 "J2" H 1250 5650 50  0000 R CNN
 F 1 "8P8C_Shielded_x4" H 1500 5550 50  0000 R CNN
 F 2 "Custom Footprints:RJ45_x4-RJSSE-5380-04" V 1150 5025 50  0001 C CNN
@@
 $EndComp
 $Comp
-L Custom_parts:8P8C_Shielded_x4 J3
+L Custom_parts:8P8C_Shielded_x4 J2
 U 3 1 5F57B5E3
 P 1150 3600
-F 0 "J3" H 1250 4250 50  0000 R CNN
+F 0 "J2" H 1250 4250 50  0000 R CNN
 F 1 "8P8C_Shielded_x4" H 1500 4150 50  0000 R CNN
 F 2 "Custom Footprints:RJ45_x4-RJSSE-5380-04" V 1150 3625 50  0001 C CNN
@@
 $EndComp
 $Comp
-L Custom_parts:8P8C_Shielded_x4 J3
+L Custom_parts:8P8C_Shielded_x4 J2
 U 2 1 5F589234
 P 7850 6150
-F 0 "J3" H 7950 6800 50  0000 R CNN
+F 0 "J2" H 7950 6800 50  0000 R CNN
 F 1 "8P8C_Shielded_x4" H 8200 6700 50  0000 R CNN
 F 2 "Custom Footprints:RJ45_x4-RJSSE-5380-04" V 7850 6175 50  0001 C CNN
@@
 $EndComp
 $Comp
-L Custom_parts:8P8C_Shielded_x4 J3
+L Custom_parts:8P8C_Shielded_x4 J2
 U 1 1 5F5922AC
 P 7850 4050
-F 0 "J3" H 7900 4700 50  0000 R CNN
+F 0 "J2" H 7900 4700 50  0000 R CNN
 F 1 "8P8C_Shielded_x4" H 8200 4600 50  0000 R CNN
 F 2 "Custom Footprints:RJ45_x4-RJSSE-5380-04" V 7850 4075 50  0001 C CNN
@@
 	-1   0    0    1
 $EndComp
-Connection ~ 3150 3000
-Wire Wire Line
-	3150 2900 3150 3000
-$Comp
-L power:GND #PWR0108
-U 1 1 61A65F9D
-P 3150 3000
-F 0 "#PWR0108" H 3150 2750 50  0001 C CNN
-F 1 "GND" H 3350 2900 50  0000 R CNN
-F 2 "" H 3150 3000 50  0001 C CNN
-F 3 "" H 3150 3000 50  0001 C CNN
-	1    3150 3000
-	1    0    0    -1
-$EndComp
-$Comp
-L Connector:Barrel_Jack_Switch J1
-U 1 1 61A65FA5
-P 2850 2900
-F 0 "J1" H 2907 3217 50  0000 C CNN
-F 1 "Barrel_Jack_Switch" H 2907 3126 50  0000 C CNN
-F 2 "Custom Footprints:DC-jack_54-00165" H 2900 2860 50  0001 C CNN
-F 3 "https://tensility.s3-us-west-2.amazonaws.com/uploads/product_doc/document/4054/54-00165.pdf" H 2900 2860 50  0001 C CNN
-F 4 "Tensility International Corp" H 2850 2900 50  0001 C CNN "Manufacturer"
-F 5 "54-00165" H 2850 2900 50  0001 C CNN "Part #"
-	1    2850 2900
-	1    0    0    -1
-$EndComp
-Text Label 3150 2800 0    50   ~ 0
-+18V
 $Comp
 L power:GND #PWR015
@@
 $EndComp
 Wire Wire Line
-	3150 2800 3450 2800
-Wire Wire Line
 	3450 2800 3850 2800
-Connection ~ 3450 2800
 $Comp
 L power:GND #PWR0102
@@
 $EndComp
 $Comp
-L Custom_parts:TC4468EOE U2
+L Custom_parts:TC4468EOE U3
 U 1 1 64F06EE9
 P 4250 3750
-F 0 "U2" H 4750 4007 60  0000 C CNN
+F 0 "U3" H 4750 4007 60  0000 C CNN
 F 1 "TC4468EOE" H 4750 3901 60  0000 C CNN
 F 2 "Custom Footprints:TC4468EOE" H 5350 3990 60  0001 C CNN
@@
 Wire Wire Line
 	5250 5950 5250 5850
-Text Label 5250 3850 0    50   ~ 0
-+18V
-Text Label 5250 5950 0    50   ~ 0
-+18V
 Wire Wire Line
 	4250 6450 4250 6550
@@
 $EndComp
 $Comp
-L Custom_parts:IRF9358TRPBF-2x_p-channel Q1
+L Custom_parts:IRF9358TRPBF-2x_p-channel Q4
 U 1 1 64F4537D
 P 7450 3000
-F 0 "Q1" H 6500 2851 60  0000 C CNN
+F 0 "Q4" H 6500 2851 60  0000 C CNN
 F 1 "IRF9358TRPBF-2x_p-channel" H 6500 2875 60  0001 C CNN
 F 2 "Custom Footprints:IRF9358TRPBF-2x_p-channel" H 6500 2815 60  0001 C CNN
@@
 Gate8
 $Comp
-L Custom_parts:IRF9358TRPBF-2x_p-channel Q2
+L Custom_parts:IRF9358TRPBF-2x_p-channel Q3
 U 1 1 64F7C414
 P 7450 4050
-F 0 "Q2" H 6500 3901 60  0000 C CNN
+F 0 "Q3" H 6500 3901 60  0000 C CNN
 F 1 "IRF9358TRPBF-2x_p-channel" H 6500 3925 60  0001 C CNN
 F 2 "Custom Footprints:IRF9358TRPBF-2x_p-channel" H 6500 3865 60  0001 C CNN
@@
 $EndComp
 $Comp
-L Custom_parts:IRF9358TRPBF-2x_p-channel Q3
+L Custom_parts:IRF9358TRPBF-2x_p-channel Q2
 U 1 1 64F7E6DD
 P 7450 5100
-F 0 "Q3" H 6500 4951 60  0000 C CNN
+F 0 "Q2" H 6500 4951 60  0000 C CNN
 F 1 "IRF9358TRPBF-2x_p-channel" H 6500 4975 60  0001 C CNN
 F 2 "Custom Footprints:IRF9358TRPBF-2x_p-channel" H 6500 4915 60  0001 C CNN
@@
 $EndComp
 $Comp
-L Custom_parts:IRF9358TRPBF-2x_p-channel Q4
+L Custom_parts:IRF9358TRPBF-2x_p-channel Q1
 U 1 1 64F81FE0
 P 7450 6150
-F 0 "Q4" H 6500 6001 60  0000 C CNN
+F 0 "Q1" H 6500 6001 60  0000 C CNN
 F 1 "IRF9358TRPBF-2x_p-channel" H 6500 6025 60  0001 C CNN
 F 2 "Custom Footprints:IRF9358TRPBF-2x_p-channel" H 6500 5965 60  0001 C CNN
@@
 $EndComp
 $Comp
-L Custom_parts:TC4468EOE U3
+L Custom_parts:TC4468EOE U2
 U 1 1 64F8812A
 P 4250 5850
-F 0 "U3" H 4750 6107 60  0000 C CNN
+F 0 "U2" H 4750 6107 60  0000 C CNN
 F 1 "TC4468EOE" H 4750 6001 60  0000 C CNN
 F 2 "Custom Footprints:TC4468EOE" H 5350 6090 60  0001 C CNN
@@
 $EndComp
 $Comp
-L Connector:Conn_01x02_Female J2
+L Connector:Conn_01x02_Female J1
 U 1 1 64F692B9
 P 2100 5300
-F 0 "J2" H 2128 5230 50  0000 L CNN
-F 1 "Conn_01x02_Female" H 2128 5185 50  0001 L CNN
-F 2 "Connector_Wire:SolderWire-0.5sqmm_1x02_P4.6mm_D0.9mm_OD2.1mm" H 2100 5300 50  0001 C CNN
-F 3 "~" H 2100 5300 50  0001 C CNN
+F 0 "J1" H 2128 5230 50  0000 L CNN
+F 1 "8P8C_Shielded_x4" H 2128 5185 50  0001 L CNN
+F 2 "Custom Footprints:RJ45_x4-RJSSE-5380-04" H 2100 5300 50  0001 C CNN
+F 3 "https://cdn.amphenol-icc.com/media/wysiwyg/files/drawing/rjsse538004.pdf" H 2100 5300 50  0001 C CNN
 	1    2100 5300
 	1    0    0    -1
 $EndComp
-$Comp
-L Device:Jumper_NO_Small JP1
-U 1 1 64FA019D
-P 1800 5300
-F 0 "JP1" H 1800 5250 50  0000 C CNN
-F 1 "Jumper_NO_Small" H 1800 5394 50  0001 C CNN
-F 2 "Jumper:SolderJumper-2_P1.3mm_Open_TrianglePad1.0x1.5mm" H 1800 5300 50  0001 C CNN
-F 3 "~" H 1800 5300 50  0001 C CNN
-	1    1800 5300
-	1    0    0    -1
-$EndComp
-Wire Wire Line
-	1700 5300 1550 5300
 Wire Wire Line
 	1900 5400 1550 5400
@@
 Wire Wire Line
 	1550 5100 2450 5100
+Wire Wire Line
+	1550 5300 1900 5300
+Text Label 3550 2800 0    50   ~ 0
+LED+
+Text Label 5250 3850 0    50   ~ 0
+LED+
+Text Label 5250 5950 0    50   ~ 0
+LED+
 $EndSCHEMATC

Commit message: Use Vin through LDO for 5V - no ext. power
This redesign uses an linear regulator to drop the Vin voltage to 5V.  This will greatly reduce the noise on the board, as well as the part count and complexity.
Parts:
- removed C1, C2: 22µF, Capacitor_SMD:C_1206_3216Metric, symbol Device:C
- removed LOGO2: Jack Polarity, Custom Footprints:Polarity_Center_Positive, symbol Graphic:Logo_Open_Hardware_Small
- removed PS1: PXO7805-500-M-TR, Custom Footprints:18V_to_5V_PXO7805-500-M-TR, symbol Custom_parts:PXO7805-500-M-TR
- added C1: 2.2uF, Custom Footprints:0508_Capacitor, symbol Device:C_Small
- added U1: NCV7805BDTRKG, Custom Footprints:12V-5V_lin_reg_NCV7805BDTRKG, symbol Custom_parts:NCV7805BDTRKG
- J1: value 8P8C_Shielded_x4 -> 2 pin header; footprint Custom Footprints:RJ45_x4-RJSSE-5380-04 -> Connector_PinSocket_2.54mm:PinSocket_1x02_P2.54mm_Vertical_SMD_Pin1Right; Manufacturer (none) -> Sullins Connector Solutions; Part # (none) -> NPTC021KFXC-RC
- renumbered C3 to C2, C4 to C3, C5 to C4, U1 to U2, U2 to U3, U3 to U4
Connections:
- net +5V: now also U1.3 (Vout)
- net GND: now also C1.1, U1.2 (GND)
- net LED+: now also C1.2, U1.1 (Vin)
Changed lines of the file:
@@
 $EndComp
 $Comp
-L Graphic:Logo_Open_Hardware_Small LOGO2
-U 1 1 5FF6ADDD
+L Graphic:Logo_Open_Hardware_Small LOGO3
+U 1 1 5FF6B1EE
 P 4550 7450
-F 0 "LOGO2" H 4550 7725 50  0001 C CNN
-F 1 "Jack Polarity" H 4300 7750 50  0000 L CNN
-F 2 "Custom Footprints:Polarity_Center_Positive" H 4550 7450 50  0001 C CNN
+F 0 "LOGO3" H 4550 7725 50  0001 C CNN
+F 1 "OSHW Logo" H 4350 7750 50  0000 L CNN
+F 2 "Symbol:OSHW-Logo2_7.3x6mm_SilkScreen" H 4550 7450 50  0001 C CNN
 F 3 "~" H 4550 7450 50  0001 C CNN
 	1    4550 7450
-	1    0    0    -1
-$EndComp
-$Comp
-L Graphic:Logo_Open_Hardware_Small LOGO3
-U 1 1 5FF6B1EE
-P 5050 7450
-F 0 "LOGO3" H 5050 7725 50  0001 C CNN
-F 1 "OSHW Logo" H 4850 7750 50  0000 L CNN
-F 2 "Symbol:OSHW-Logo2_7.3x6mm_SilkScreen" H 5050 7450 50  0001 C CNN
-F 3 "~" H 5050 7450 50  0001 C CNN
-	1    5050 7450
 	1    0    0    -1
 $EndComp
@@
 Text Label 7450 6450 2    50   ~ 0
 LED8+
-$Comp
-L Custom_parts:PXO7805-500-M-TR PS1
-U 1 1 64EDC858
-P 4150 2850
-F 0 "PS1" H 4175 3115 50  0000 C CNN
-F 1 "PXO7805-500-M-TR" H 4175 3024 50  0000 C CNN
-F 2 "Custom Footprints:18V_to_5V_PXO7805-500-M-TR" H 3650 2550 50  0001 L BNN
-F 3 "https://www.cui.com/product/resource/pxo78-500-m.pdf" H 4250 2850 50  0001 L BNN
-F 4 "CUI Inc." H 4150 2850 50  0001 C CNN "Manufacturer"
-F 5 "PXO7805-500-M-TR" H 4150 2850 50  0001 C CNN "Part #"
-	1    4150 2850
-	1    0    0    -1
-$EndComp
-Text Label 4500 2800 0    50   ~ 0
+Text Label 4650 2800 0    50   ~ 0
 +5V
 $Comp
 L power:GND #PWR0101
 U 1 1 64EE383E
-P 3450 3100
-F 0 "#PWR0101" H 3450 2850 50  0001 C CNN
-F 1 "GND" H 3650 3000 50  0000 R CNN
-F 2 "" H 3450 3100 50  0001 C CNN
-F 3 "" H 3450 3100 50  0001 C CNN
-	1    3450 3100
-	1    0    0    -1
-$EndComp
-$Comp
-L power:GND #PWR0103
-U 1 1 64EE65BC
-P 3850 2900
-F 0 "#PWR0103" H 3850 2650 50  0001 C CNN
-F 1 "GND" H 4050 2800 50  0000 R CNN
-F 2 "" H 3850 2900 50  0001 C CNN
-F 3 "" H 3850 2900 50  0001 C CNN
-	1    3850 2900
-	1    0    0    -1
-$EndComp
-$Comp
-L Device:C C2
-U 1 1 64EE98B9
-P 4650 2950
-F 0 "C2" H 4765 2996 50  0000 L CNN
-F 1 "22µF" H 4765 2905 50  0000 L CNN
-F 2 "Capacitor_SMD:C_1206_3216Metric" H 4688 2800 50  0001 C CNN
-F 3 "https://product.tdk.com/system/files/dam/doc/product/capacitor/ceramic/mlcc/catalog/mlcc_commercial_general_en.pdf" H 4650 2950 50  0001 C CNN
-F 4 "TDK Corporation" H 4650 2950 50  0001 C CNN "Manufacturer"
-F 5 "C3216X5R1V226M160AC" H 4650 2950 50  0001 C CNN "Part #"
-	1    4650 2950
+P 4050 3000
+F 0 "#PWR0101" H 4050 2750 50  0001 C CNN
+F 1 "GND" H 4250 2900 50  0000 R CNN
+F 2 "" H 4050 3000 50  0001 C CNN
+F 3 "" H 4050 3000 50  0001 C CNN
+	1    4050 3000
 	1    0    0    -1
 $EndComp
@@
 L power:GND #PWR0104
 U 1 1 64EE98BF
-P 4650 3100
-F 0 "#PWR0104" H 4650 2850 50  0001 C CNN
-F 1 "GND" H 4850 3000 50  0000 R CNN
-F 2 "" H 4650 3100 50  0001 C CNN
-F 3 "" H 4650 3100 50  0001 C CNN
-	1    4650 3100
-	1    0    0    -1
-$EndComp
-Wire Wire Line
-	4500 2800 4650 2800
-$Comp
-L Device:C C1
-U 1 1 64EEB8D5
-P 3450 2950
-F 0 "C1" H 3565 2996 50  0000 L CNN
-F 1 "22µF" H 3565 2905 50  0000 L CNN
-F 2 "Capacitor_SMD:C_1206_3216Metric" H 3488 2800 50  0001 C CNN
-F 3 "https://product.tdk.com/system/files/dam/doc/product/capacitor/ceramic/mlcc/catalog/mlcc_commercial_general_en.pdf" H 3450 2950 50  0001 C CNN
-F 4 "TDK Corporation" H 3450 2950 50  0001 C CNN "Manufacturer"
-F 5 "C3216X5R1V226M160AC" H 3450 2950 50  0001 C CNN "Part #"
-	1    3450 2950
-	1    0    0    -1
-$EndComp
-Wire Wire Line
-	3450 2800 3850 2800
+P 4350 3150
+F 0 "#PWR0104" H 4350 2900 50  0001 C CNN
+F 1 "GND" H 4550 3050 50  0000 R CNN
+F 2 "" H 4350 3150 50  0001 C CNN
+F 3 "" H 4350 3150 50  0001 C CNN
+	1    4350 3150
+	1    0    0    -1
+$EndComp
 $Comp
 L power:GND #PWR0102
@@
 $EndComp
 $Comp
-L Device:C_Small C4
+L Device:C_Small C3
 U 1 1 61940B33
 P 5250 3650
-F 0 "C4" V 5450 3600 50  0000 L CNN
+F 0 "C3" V 5450 3600 50  0000 L CNN
 F 1 "2.2uF" V 5350 3550 50  0000 L CNN
 F 2 "Custom Footprints:0508_Capacitor" H 5250 3650 50  0001 C CNN
@@
 $EndComp
 $Comp
-L Custom_parts:TC4468EOE U3
+L Custom_parts:TC4468EOE U4
 U 1 1 64F06EE9
 P 4250 3750
-F 0 "U3" H 4750 4007 60  0000 C CNN
+F 0 "U4" H 4750 4007 60  0000 C CNN
 F 1 "TC4468EOE" H 4750 3901 60  0000 C CNN
 F 2 "Custom Footprints:TC4468EOE" H 5350 3990 60  0001 C CNN
@@
 $EndComp
 $Comp
-L Device:C_Small C5
+L Device:C_Small C4
 U 1 1 64F08194
 P 5250 5750
-F 0 "C5" V 5450 5700 50  0000 L CNN
+F 0 "C4" V 5450 5700 50  0000 L CNN
 F 1 "2.2uF" V 5350 5650 50  0000 L CNN
 F 2 "Custom Footprints:0508_Capacitor" H 5250 5750 50  0001 C CNN
@@
 	5250 6450 5250 6550
 $Comp
-L Custom_parts:SN74LV138AT_D_16 U1
+L Custom_parts:SN74LV138AT_D_16 U2
 U 1 1 64FF7275
 P 2700 4800
-F 0 "U1" H 3200 5057 60  0000 C CNN
+F 0 "U2" H 3200 5057 60  0000 C CNN
 F 1 "SN74LV138AT_D_16" H 3200 4951 60  0000 C CNN
 F 2 "Custom Footprints:SN74LV138ATD" H 3800 5040 60  0001 C CNN
@@
 $EndComp
 $Comp
-L Device:C_Small C3
+L Device:C_Small C2
 U 1 1 65045290
 P 3700 4600
-F 0 "C3" V 3900 4550 50  0000 L CNN
+F 0 "C2" V 3900 4550 50  0000 L CNN
 F 1 "2.2uF" V 3800 4500 50  0000 L CNN
 F 2 "Custom Footprints:0508_Capacitor" H 3700 4600 50  0001 C CNN
@@
 $EndComp
 $Comp
-L Custom_parts:TC4468EOE U2
+L Custom_parts:TC4468EOE U3
 U 1 1 64F8812A
 P 4250 5850
-F 0 "U2" H 4750 6107 60  0000 C CNN
+F 0 "U3" H 4750 6107 60  0000 C CNN
 F 1 "TC4468EOE" H 4750 6001 60  0000 C CNN
 F 2 "Custom Footprints:TC4468EOE" H 5350 6090 60  0001 C CNN
@@
 P 2100 5300
 F 0 "J1" H 2128 5230 50  0000 L CNN
-F 1 "8P8C_Shielded_x4" H 2128 5185 50  0001 L CNN
-F 2 "Custom Footprints:RJ45_x4-RJSSE-5380-04" H 2100 5300 50  0001 C CNN
-F 3 "https://cdn.amphenol-icc.com/media/wysiwyg/files/drawing/rjsse538004.pdf" H 2100 5300 50  0001 C CNN
+F 1 "2 pin header" H 2128 5185 50  0001 L CNN
+F 2 "Connector_PinSocket_2.54mm:PinSocket_1x02_P2.54mm_Vertical_SMD_Pin1Right" H 2100 5300 50  0001 C CNN
+F 3 "https://mm.digikey.com/Volume0/opasdata/d220001/medias/docus/2900/NPxCxx1KFXx-RC%2010487-D.pdf" H 2100 5300 50  0001 C CNN
+F 4 "Sullins Connector Solutions" H 2100 5300 50  0001 C CNN "Manufacturer"
+F 5 "NPTC021KFXC-RC" H 2100 5300 50  0001 C CNN "Part #"
 	1    2100 5300
 	1    0    0    -1
@@
 Wire Wire Line
 	1550 5300 1900 5300
-Text Label 3550 2800 0    50   ~ 0
+Text Label 4050 2800 2    50   ~ 0
 LED+
 Text Label 5250 3850 0    50   ~ 0
@@
 Text Label 5250 5950 0    50   ~ 0
 LED+
+$Comp
+L Device:C_Small C1
+U 1 1 65365726
+P 4050 2900
+F 0 "C1" H 4150 2850 50  0000 L CNN
+F 1 "2.2uF" H 4150 2950 50  0000 L CNN
+F 2 "Custom Footprints:0508_Capacitor" H 4050 2900 50  0001 C CNN
+F 3 "https://ds.yuden.co.jp/TYCOMPAS/ut/detail?pn=TWK212B7225MD-T%20&u=M" H 4050 2900 50  0001 C CNN
+F 4 "Taiyo Yuden" H 4050 2900 50  0001 C CNN "Manufacturer"
+F 5 "TWK212B7225MD-T" H 4050 2900 50  0001 C CNN "Part #"
+	1    4050 2900
+	-1   0    0    1
+$EndComp
+$Comp
+L Custom_parts:NCV7805BDTRKG U1
+U 1 1 65367633
+P 3850 2800
+F 0 "U1" H 4350 3057 60  0000 C CNN
+F 1 "NCV7805BDTRKG" H 4350 2951 60  0000 C CNN
+F 2 "Custom Footprints:12V-5V_lin_reg_NCV7805BDTRKG" H 4750 3040 60  0001 C CNN
+F 3 "https://www.onsemi.com/pdf/datasheet/mc7800-d.pdf" H 4350 2951 60  0001 C CNN
+F 4 "onsemi" H 3850 2800 50  0001 C CNN "Manufacturer"
+F 5 "NCV7805BDTRKG" H 3850 2800 50  0001 C CNN "Part #"
+	1    3850 2800
+	1    0    0    -1
+$EndComp
 $EndSCHEMATC
