File: LED Driver 1x8 Mux.kicad_pcb (KiCad board)
At the start: 2 copper layers, 117 x 72.4 mm, 20 parts, among them J1 2 pin header, J2 8P8C_Shielded_x4, Q1 SO8_IRF9358TRPBF_INF, Q2 SO8_IRF9358TRPBF_INF, Q3 SO8_IRF9358TRPBF_INF, Q4 SO8_IRF9358TRPBF_INF, U1 NCV7805BDTRKG, U2 SN74LV138AT_D_16, U3 SOIC16-W_MC_MCH, U4 SOIC16-W_MC_MCH

Commit message: Change name
Parts:
- Q1, Q2, Q3, Q4: value SO8_IRF9358TRPBF_INF -> IRF9358TRPBF-2x_p-channel
Routing:
- net GND: vias 229 -> 231

Commit message: Update naming on board
Other:
- board text added: "Designed by: Benjamin E. Smith Funded by: NIH P30EY003176 https://github.com/Llamero/LED_Driver_1x8_Mux"
- board text removed: "Designed by: Benjamin E. Smith Funded by: NIH P30EY003176 https://github.com/Llamero/High_speed_1x8_LED_mux"
